Commit message: URDF refactoring for some sensors

File: ca_description/urdf/create_2.urdf.xacro (robot description, xacro)
@@ -7,4 +7,4 @@
   </xacro:create_base>
   <!-- Roomblock -->
-  <xacro:roomblock visualize="$(arg visualize)"/>
+  <xacro:roomblock parent="base_link" visualize="$(arg visualize)"/>
 </robot>

File: ca_description/urdf/create_base_gazebo.urdf.xacro (robot description, xacro)
@@ -30,8 +30,7 @@
         <topicName>gts</topicName>
         <gaussianNoise>0</gaussianNoise>
-        <frameName>world</frameName>
+        <frameName>map</frameName>
         <xyzOffsets>0 0 0</xyzOffsets>
         <rpyOffsets>0 0 0</rpyOffsets>
-        <!--<interface:position name="p3d_base_position"/>-->
       </plugin>
     </gazebo>

File: ca_description/urdf/roomblock.urdf.xacro (robot description, xacro)
@@ -4,41 +4,28 @@
 -->
 <robot xmlns:xacro="http://ros.org/wiki/xacro">
-  <xacro:include filename="$(find ca_description)/urdf/roomblock_gazebo.urdf.xacro"/>
-  <xacro:property name="block_z_offset" value="0.061"/>
-  <xacro:property name="laser_z_offset" value="0.1308"/>
-  <xacro:property name="camera_x_offset" value="0.04"/>
-  <xacro:property name="camera_z_offset" value="0.1"/>
-  <material name="Grey">
-    <color rgba="0.2 0.2 0.2 1.0"/>
-  </material>
-  <xacro:macro name="roomblock" params="visualize:=false">
+  <xacro:include filename="$(find ca_description)/urdf/common_properties.xacro"/>
+  <xacro:include filename="$(find ca_description)/urdf/roomblock_gazebo.xacro"/>
+  <xacro:include filename="$(find ca_description)/urdf/sensors/laser_sensor.xacro"/>
+  <xacro:include filename="$(find ca_description)/urdf/sensors/camera_sensor.xacro"/>
+  <xacro:macro name="roomblock" params="parent visualize:=false">
+    <xacro:property name="z" value="0.061"/>
+    <xacro:property name="roomblock_link" value="block_link"/>
+    <xacro:property name="parent_link" value="${parent}"/>
     <joint name="block_joint" type="fixed">
-      <origin xyz="0 0 ${block_z_offset}" rpy="0 0 0" />
-      <parent link="base_link"/>
-      <child link="block_link" />
+      <origin xyz="0 0 ${z}" rpy="0 0 0" />
+      <parent link="${parent_link}"/>
+      <child link="${roomblock_link}" />
     </joint>
-    <link name="block_link">
+    <link name="${roomblock_link}">
       <visual>
-        <origin xyz="0 0 0" rpy="0 0 0" />
         <geometry>
-  	<mesh filename="package://ca_description/meshes/block.dae"/>
+  	       <mesh filename="package://ca_description/meshes/block.dae"/>
         </geometry>
         <material name="Grey" />
       </visual>
     </link>
-    <joint name="laser_joint" type="fixed">
-      <origin xyz="0 0 ${laser_z_offset}" rpy="0 0 ${pi}" />
-      <parent link="block_link" />
-      <child link="laser_link" />
-    </joint>
-    <link name="laser_link"/>
-    <joint name="camera_joint" type="fixed">
-      <origin xyz="${camera_x_offset} 0 ${camera_z_offset}" rpy="0 0 0" />
-      <parent link="block_link" />
-      <child link="raspicam_link" />
-    </joint>
-    <link name="raspicam_link"/>
-    <!-- Gazebo properties -->
-    <xacro:roomblock_gazebo visualize="$(arg visualize)"/>
+    <xacro:laser_sensor parent="${roomblock_link}" visualize="$(arg visualize)"/>
+    <xacro:camera_sensor parent="${roomblock_link}"/>
+    <xacro:roomblock_gazebo link_name="${roomblock_link}"/>
   </xacro:macro>
 </robot>
