Commit message: Some fixes

File: ca_description/urdf/create_base_gazebo.urdf.xacro (robot description, xacro)
@@ -3,4 +3,5 @@
   <xacro:macro name="sim_create_base">
     <gazebo>
+      <!-- Diff-drive controller -->
       <plugin name="differential_drive_controller" filename="libgazebo_ros_diff_drive.so">
         <alwaysOn>true</alwaysOn>
@@ -24,4 +25,5 @@
         <publishTf>1</publishTf>
       </plugin>
+      <!-- Ground truth -->
       <plugin name="p3d_base_controller" filename="libgazebo_ros_p3d.so">
         <alwaysOn>true</alwaysOn>
@@ -35,4 +37,24 @@
       </plugin>
     </gazebo>
+    <!-- Bumpers -->
+    <gazebo reference="base_link">
+      <gravity>true</gravity>
+      <self_collide>false</self_collide>
+      <sensor name='bumper_contact_sensor' type='contact'>
+        <always_on>true</always_on>
+        <update_rate>50</update_rate>
+        <contact>
+          <collision>base_link_collision</collision>
+          <topic>bumpers</topic>
+        </contact>
+        <!-- Plugin -->
+        <!-- <plugin name="gazebo_ros_bumper_controller" filename="libgazebo_ros_bumper.so">
+          <frameName>base_link</frameName>
+          <bumperTopicName>bumper</bumperTopicName>
+        </plugin> -->
+        <!-- <plugin name="gazebo_ros_bumper_controller" filename="libcreate_bumper_plugin.so"/> -->
+      </sensor>
+    </gazebo>
+    <!-- Wheels -->
     <gazebo reference="left_wheel_link">
       <mu1>1.0</mu1>
@@ -51,20 +73,4 @@
       <maxVel>1.0</maxVel>
     </gazebo>
-    <gazebo reference="rear_wheel_link">
-      <mu1>0.0</mu1>
-      <mu2>0.0</mu2>
-      <kp>1000000.0</kp>
-      <kd>100.0</kd>
-      <minDepth>0.001</minDepth>
-      <maxVel>1.0</maxVel>
-    </gazebo>
-    <gazebo reference="front_wheel_link">
-      <mu1>0.0</mu1>
-      <mu2>0.0</mu2>
-      <kp>1000000.0</kp>
-      <kd>100.0</kd>
-      <minDepth>0.001</minDepth>
-      <maxVel>1.0</maxVel>
-    </gazebo>
   </xacro:macro>
 </robot>

File: ca_description/urdf/sensors/imu_sensor.xacro (robot description, xacro)
@@ -8,5 +8,5 @@
   <xacro:property name="x" value="0"/>
   <xacro:property name="y" value="-0.04"/>
-  <xacro:property name="z" value="0.1"/>
+  <xacro:property name="z" value="0.13"/>
   <xacro:property name="R" value="0"/>
   <xacro:property name="P" value="0"/>
@@ -21,5 +21,5 @@
     <xacro:dummy_inertia/>
   </link>
-  <xacro:sim_imu/>
+  <xacro:imu_sensor_gazebo/>
 </xacro:macro>
 </robot>

File: ca_description/urdf/sensors/imu_sensor_gazebo.xacro (robot description, xacro)
@@ -1,5 +1,5 @@
 <?xml version="1.0" ?>
 <robot xmlns:xacro="http://ros.org/wiki/xacro">
-<xacro:macro name="sim_imu">
+<xacro:macro name="imu_sensor_gazebo">
   <gazebo>
     <plugin name="imu_controller" filename="libgazebo_ros_imu.so">
