Commit message: Pre course fixes (#18)
* Using variable instead of default name

* Fix inertias

* Fix LegacyMode again

* Support initial pose for AMCL

* Fix RViz config for navigation

* Add slam_gmapping example

* Fix RViz launchfile

* Use optical link for camera

* Fix position of slam_gmapping launchfile and use config YAML

* Use HTTPS instead of SSH

* Clean up and improve XACRO model

File: ca_description/urdf/create_base_gazebo.xacro (robot description, xacro)
@@ -2,4 +2,7 @@
 <robot xmlns:xacro="http://ros.org/wiki/xacro">
   <xacro:macro name="sim_create_base">
+    <xacro:property name="diffdrive_update_rate" value="40"/>
+    <xacro:property name="wheel_torque" value="0.5"/>
+    <xacro:property name="wheel_accel" value="0.5"/>
     <gazebo>
       <!-- Diff-drive controller -->
@@ -8,6 +11,6 @@
         <rosDebugLevel>na</rosDebugLevel>
         <updateRate>${diffdrive_update_rate}</updateRate>
-        <leftJoint>right_wheel_joint</leftJoint>
-        <rightJoint>left_wheel_joint</rightJoint>
+        <leftJoint>left_wheel_joint</leftJoint>
+        <rightJoint>right_wheel_joint</rightJoint>
         <wheelSeparation>${wheel_separation}</wheelSeparation>
         <wheelDiameter>${wheel_radius * 2}</wheelDiameter>
@@ -28,5 +31,5 @@
       <plugin name="p3d_base_controller" filename="libgazebo_ros_p3d.so">
         <alwaysOn>true</alwaysOn>
-        <updateRate>100.0</updateRate>
+        <updateRate>60.0</updateRate>
         <bodyName>base_link</bodyName>
         <topicName>gts</topicName>
