Commit message: Add Turtlebot stack and lots of lasers (#142)
* Edit roomblock

* Create specific RPLidar Xacro

* WIP: Add other sensors

* Set parent for cliff sensors

* WIP

* Clean up URDFs

* More updates

* Fixed a lot of things

* Improve turtlebot.xacro

* Fix sensors in roomblock stack

* Simplify code using a .yaml to define poses

* Rename and cleaned up meshes

* Fix wrong default laser

* Fix Lidar error

* Improve Turtlebot stack

* Move sensor meshes to 'sensors' folder

* Use turtlebot stack by default

* Use meshes from new directory

* Improve calling of stacks

* Add Nvidia Jetson Nano

File: ca_description/urdf/create_2.xacro (robot description, xacro)
@@ -2,5 +2,4 @@
 <robot name="create_2" xmlns:xacro="http://ros.org/wiki/xacro">
   <xacro:include filename="$(find ca_description)/urdf/create_base.xacro"/>
-  <xacro:include filename="$(find ca_description)/urdf/roomblock.xacro"/>
   <xacro:property name="robot_name" value="$(arg robot_name)"/>
   <xacro:property name="wheel_separation" value="0.235"/>
@@ -15,5 +14,9 @@
     <mesh filename="package://ca_description/meshes/create_2.dae" />
   </xacro:create_base>
-  <!-- Roomblock -->
-  <xacro:roomblock parent="base_link" visualize="$(arg visualize)"/>
+  <!-- Stacks -->
+  <xacro:property name="stack" value="$(arg stack)"/>
+  <xacro:property name="stack_yaml" value="$(find ca_description)/urdf/stacks/poses.yaml"/>
+  <xacro:property name="stack_dict" value="${load_yaml(stack_yaml)}"/>
+  <xacro:property name="stack_origin" value="${stack_dict[stack]}"/>
+  <xacro:include filename="$(find ca_description)/urdf/stacks/${stack}.xacro"/>
 </robot>

File: ca_description/urdf/create_base.xacro (robot description, xacro)
@@ -1,12 +1,13 @@
 <?xml version="1.0" ?>
 <robot xmlns:xacro="http://ros.org/wiki/xacro">
+  <xacro:include filename="$(find ca_description)/urdf/common_properties.xacro"/>
+  <xacro:include filename="$(find ca_description)/urdf/create_base_gazebo.xacro"/>
+  <xacro:include filename="$(find ca_description)/urdf/create_caster_wheel.xacro"/>
+  <xacro:include filename="$(find ca_description)/urdf/create_wheel.xacro"/>
+  <xacro:include filename="$(find ca_description)/urdf/sensors/imu_sensor.xacro"/>
+  <xacro:include filename="$(find ca_description)/urdf/sensors/wall_sensor.xacro"/>
+  <xacro:include filename="$(find ca_description)/urdf/sensors/cliff_sensors.xacro"/>
+  <xacro:include filename="$(find ca_description)/urdf/sensors/omni_sensor.xacro"/>
   <xacro:macro name="create_base" params="wheel_separation wheel_radius wheel_width base_diameter *mesh visualize:=false">
-    <xacro:include filename="$(find ca_description)/urdf/create_base_gazebo.xacro"/>
-    <xacro:include filename="$(find ca_description)/urdf/create_caster_wheel.xacro"/>
-    <xacro:include filename="$(find ca_description)/urdf/create_wheel.xacro"/>
-    <xacro:include filename="$(find ca_description)/urdf/sensors/imu_sensor.xacro"/>
-    <xacro:include filename="$(find ca_description)/urdf/sensors/wall_sensor.xacro"/>
-    <xacro:include filename="$(find ca_description)/urdf/sensors/cliff_sensors.xacro"/>
-    <xacro:include filename="$(find ca_description)/urdf/sensors/omni_sensor.xacro"/>
     <xacro:property name="base_link_offset_z" value="0.0308"/>
     <xacro:property name="base_offset_z" value="0.017"/>
@@ -45,26 +46,34 @@
       </collision>
     </link>
-    <xacro:wall_sensor visualize="${visualize}"/>
-    <xacro:cliff_sensor name="side_left">
+    <xacro:wall_sensor visualize="${visualize}">
+      <origin xyz="0.09 -0.12 0.042" rpy="0 0 -1"/>
+    </xacro:wall_sensor>
+    <xacro:cliff_sensor name="side_left_cliff_sensor">
       <origin xyz="0.07 0.14 0.01" rpy="0 ${pi/2 - 0.09} 0" />
     </xacro:cliff_sensor>
-    <xacro:cliff_sensor name="side_right">
+    <xacro:cliff_sensor name="side_right_cliff_sensor">
       <origin xyz="0.07 -0.14 0.01" rpy="0 ${pi/2 - 0.09} 0" />
     </xacro:cliff_sensor>
-    <xacro:cliff_sensor name="front_left">
+    <xacro:cliff_sensor name="front_left_cliff_sensor">
       <origin xyz="0.15 0.04 0.01" rpy="0 ${pi/2 - 0.09} 0" />
     </xacro:cliff_sensor>
-    <xacro:cliff_sensor name="front_right">
+    <xacro:cliff_sensor name="front_right_cliff_sensor">
       <origin xyz="0.15 -0.04 0.01" rpy="0 ${pi/2 - 0.09} 0" />
     </xacro:cliff_sensor>
     <xacro:imu_sensor name="imu">
-      <origin xyz="0 -0.04 0.13" rpy="0 0 0"/>
+      <origin xyz="0 -0.04 0.13"/>
     </xacro:imu_sensor>
-    <xacro:omni_sensor name="omni_sensor" diameter="0.1">
-      <origin xyz="0.145 0 ${base_link_offset_z}" rpy="0 0 0"/>
+    <xacro:omni_sensor diameter="0.1">
+      <origin xyz="0.145 0 ${base_link_offset_z}"/>
     </xacro:omni_sensor>
-    <xacro:create_wheel prefix="left" y_offset="${wheel_separation / 2}" wheel_radius="${wheel_radius}" wheel_width="${wheel_width}"/>
-    <xacro:create_wheel prefix="right" y_offset="${wheel_separation / -2}" wheel_radius="${wheel_radius}" wheel_width="${wheel_width}"/>
-    <xacro:caster_wheel/>
+    <xacro:wheel name="wheel_left" radius="${wheel_radius}" width="${wheel_width}">
+      <origin xyz="0 ${wheel_separation/2} 0.015" rpy="0 ${pi/2} ${pi/2}"/>
+    </xacro:wheel>
+    <xacro:wheel name="wheel_right" radius="${wheel_radius}" width="${wheel_width}">
+      <origin xyz="0 ${-wheel_separation/2} 0.015" rpy="0 ${pi/2} ${pi/2}"/>
+    </xacro:wheel>
+    <xacro:caster_wheel>
+      <origin xyz="0.13 0 0"/>
+    </xacro:caster_wheel>
     <!-- Simulation sensors -->
     <xacro:sim_create_base/>

File: ca_description/urdf/sensors/cliff_sensors.xacro (robot description, xacro)
@@ -1,15 +1,45 @@
 <?xml version="1.0" ?>
 <robot xmlns:xacro="http://ros.org/wiki/xacro">
-<xacro:macro name="cliff_sensor" params="name *origin visualize:=false">
+<xacro:macro name="cliff_sensor" params="name:=cliff_sensor parent:=base_link *origin visualize:=false">
   <xacro:include filename="$(find ca_description)/urdf/common_properties.xacro"/>
-  <xacro:include filename="$(find ca_description)/urdf/sensors/cliff_sensors_gazebo.xacro"/>
-  <xacro:property name="parent_link" value="base_link"/>
-  <joint name="${name}_cliff_sensor_joint" type="fixed">
+  <xacro:property name="parent_link"        value="${parent}"/>
+  <xacro:property name="link_name"          value="${name}_link"/>
+  <xacro:property name="min_range_m"        value="0.01"/>
+  <xacro:property name="max_range_m"        value="0.04"/>
+  <xacro:property name="rate_hz"            value="20.0"/>
+  <xacro:property name="min_cliff_value_cm" value="3.85"/>
+  <joint name="${name}_joint" type="fixed">
     <xacro:insert_block name="origin" />
     <parent link="${parent_link}" />
-    <child link="${name}_cliff_sensor_link" />
+    <child link="${link_name}" />
   </joint>
-  <link name="${name}_cliff_sensor_link" />
-  <xacro:cliff_plugin visualize="${visualize}" name="${name}"/>
+  <link name="${link_name}" />
+  <gazebo reference="${link_name}">
+    <sensor type="ray" name="${name}_sensor">
+      <always_on>true</always_on>
+      <update_rate>${rate_hz}</update_rate>
+      <visualize>${visualize}</visualize>
+      <ray>
+        <scan>
+          <horizontal>
+            <samples>1</samples>
+            <resolution>1</resolution>
+            <min_angle>0</min_angle>
+            <max_angle>0</max_angle>
+          </horizontal>
+        </scan>
+        <range>
+          <min>${min_range_m}</min>
+          <max>${max_range_m}</max>
+          <resolution>0.1</resolution>
+        </range>
+      </ray>
+      <plugin name="gazebo_ros_${name}" filename="libcreate_cliff_plugin.so">
+        <topicName>${name}/raw</topicName>
+        <frameName>${link_name}</frameName>
+        <cliffValue>${min_cliff_value_cm*cm_to_meters}</cliffValue>
+      </plugin>
+    </sensor>
+  </gazebo>
 </xacro:macro>
 </robot>

File: ca_description/urdf/sensors/imu_sensor.xacro (robot description, xacro)
@@ -1,8 +1,7 @@
 <?xml version="1.0" ?>
 <robot xmlns:xacro="http://ros.org/wiki/xacro">
-<xacro:macro name="imu_sensor" params="name *origin">
+<xacro:macro name="imu_sensor" params="name:=imu_sensor parent:=base_link *origin">
   <xacro:include filename="$(find ca_description)/urdf/common_properties.xacro"/>
-  <xacro:include filename="$(find ca_description)/urdf/sensors/imu_sensor_gazebo.xacro"/>
-  <xacro:property name="parent_link" value="base_link"/>
+  <xacro:property name="parent_link" value="${parent}"/>
   <xacro:property name="link_name" value="${name}_link"/>
   <joint name="${name}_joint" type="fixed">
@@ -11,8 +10,17 @@
     <child link="${link_name}" />
   </joint>
-  <link name="${link_name}">
-    <xacro:dummy_inertia/>
-  </link>
-  <xacro:imu_sensor_gazebo name="${name}" link_name="${link_name}"/>
+  <link name="${link_name}"/>
+  <gazebo>
+    <plugin name="${name}" filename="libgazebo_ros_imu.so">
+      <alwaysOn>true</alwaysOn>
+      <updateRate>30</updateRate>
+      <bodyName>${link_name}</bodyName>
+      <topicName>${name}/data</topicName>
+      <serviceName>${name}/is_calibrated</serviceName>
+      <gaussianNoise>${0.0017*0.0017}</gaussianNoise>
+      <xyzOffsets>0 0 0</xyzOffsets>
+      <rpyOffsets>0 0 0</rpyOffsets>
+    </plugin>
+  </gazebo>
 </xacro:macro>
 </robot>
