Commit message: Cliff sensor plugin (#136)
* Create a cliff plugin

Changed the plugin from the simulation to now publish a boolean

Addressed all the comments

Fixed the xacro name issues

Added passing the number of the robot via launch-file

Added functional cliff msg publisher

Fixed minor issues

Addressed most of the comments

Addressed the create_cliff comments

Changed the xacro fails to avoid repetition

Modified the SMACH to work with the cliff message

Modified the rosnode to use as a smartpointer

Addressed the xacro comments

Changed the cliff variables to work with a dictionary

fixup! Changed the cliff variables to work with a dictionary

* Fix linter

* Add missing dependencies

* Do some modifications

Co-authored-by: Steven Desvars <53347092+stevendes@users.noreply.github.com>

File: ca_description/urdf/sensors/cliff_sensors.xacro (robot description, xacro)
@@ -1,45 +1,15 @@
 <?xml version="1.0" ?>
 <robot xmlns:xacro="http://ros.org/wiki/xacro">
-<xacro:macro name="cliff_sensors" params="visualize:=false">
+<xacro:macro name="cliff_sensor" params="name *origin visualize:=false">
   <xacro:include filename="$(find ca_description)/urdf/common_properties.xacro"/>
   <xacro:include filename="$(find ca_description)/urdf/sensors/cliff_sensors_gazebo.xacro"/>
   <xacro:property name="parent_link" value="base_link"/>
-  <xacro:property name="name_side_left" value="side_left"/>
-  <xacro:property name="name_side_right" value="side_right"/>
-  <xacro:property name="name_front_left" value="front_left"/>
-  <xacro:property name="name_front_right" value="front_right"/>
-  <joint name="${name_side_left}_cliff_sensor_joint" type="fixed">
-    <origin xyz="0.07 0.14 0.01" rpy="0 ${pi/2} 0" />
+  <joint name="${name}_cliff_sensor_joint" type="fixed">
+    <xacro:insert_block name="origin" />
     <parent link="${parent_link}" />
-    <child link="${name_side_left}_cliff_sensor_link" />
+    <child link="${name}_cliff_sensor_link" />
   </joint>
-  <joint name="${name_side_right}_cliff_sensor_joint" type="fixed">
-    <origin xyz="0.07 -0.14 0.01" rpy="0 ${pi/2} 0" />
-    <parent link="${parent_link}" />
-    <child link="${name_side_right}_cliff_sensor_link" />
-  </joint>
-  <joint name="${name_front_left}_front_cliff_sensor_joint" type="fixed">
-    <origin xyz="0.15 0.04 0.01" rpy="0 ${pi/2} 0" />
-    <parent link="${parent_link}" />
-    <child link="${name_front_left}_cliff_sensor_link" />
-  </joint>
-  <joint name="${name_front_right}_cliff_sensor_joint" type="fixed">
-    <origin xyz="0.15 -0.04 0.01" rpy="0 ${pi/2} 0" />
-    <parent link="${parent_link}" />
-    <child link="${name_front_right}_cliff_sensor_link" />
-  </joint>
-  <link name="${name_side_left}_cliff_sensor_link">
-    <xacro:dummy_inertia/>
-  </link>
-  <link name="${name_side_right}_cliff_sensor_link">
-    <xacro:dummy_inertia/>
-  </link>
-  <link name="${name_front_left}_cliff_sensor_link">
-    <xacro:dummy_inertia/>
-  </link>
-  <link name="${name_front_right}_cliff_sensor_link">
-    <xacro:dummy_inertia/>
-  </link>
-  <xacro:sim_create_cliff_sensors visualize="${visualize}"/>
+  <link name="${name}_cliff_sensor_link" />
+  <xacro:cliff_plugin visualize="${visualize}" name="${name}"/>
 </xacro:macro>
 </robot>
