Commit message: Edit robot_description with IMU position

File: ca_description/urdf/sensors/imu_sensor.xacro (robot description, xacro)
@@ -7,6 +7,6 @@
   <xacro:property name="link_name" value="gyro_link"/>
   <xacro:property name="x" value="0"/>
-  <xacro:property name="y" value="0"/>
-  <xacro:property name="z" value="0.04"/>
+  <xacro:property name="y" value="-0.04"/>
+  <xacro:property name="z" value="0.1"/>
   <xacro:property name="R" value="0"/>
   <xacro:property name="P" value="0"/>

Commit message: Change IMU position in robot_description

File: ca_description/urdf/sensors/imu_sensor.xacro (robot description, xacro)
@@ -13,5 +13,5 @@
   <xacro:property name="Y" value="0"/>
   <joint name="gyro_joint" type="fixed">
-    <axis xyz="0 1 0" />
+    <axis xyz="1 0 0" />
     <origin xyz="${x} ${y} ${z}" rpy="${R} ${P} ${Y}"/>
     <parent link="${parent_link}" />

Commit message: Add real IMU (#209)
* Update ca_imu package

* Install RTIMULib dependency in Docker

* Add MPU9255

* Update installation docs

* Add i2c_imu to installation

* Fix Travis installation

* Fix tf_prefix

* Test Travis

* Change IMU rate to: compass * 2 = accel

* Add debug nodes

* Add new frame to IMU

* Fix IMU!

* Remove IMU config

* More fixes

* Fix remap

* Last fix

* Details

* Fix OGL in Travis

* Delete imu_transformer

* Don't install RTIMULib automatically

* Update Travis

* Travis again

* Fix IMU topic for Gazebo

* Fix linter

* Update README

File: ca_description/urdf/sensors/imu_sensor.xacro (robot description, xacro)
@@ -18,4 +18,7 @@
     </visual>
   </link>
+  <gazebo reference="${link_name}">
+    <material>Gazebo/BlueGlow</material>
+  </gazebo>
   <gazebo>
     <plugin name="${name}" filename="libgazebo_ros_imu.so">
