Commit message: Fix Tf for 3D cameras (#177)
* Add missing textures

* Don't publish Tf for real camera

* Use optical frame as plugin frame

* Fix Tf for 3D cameras

* fixup! Fix Tf for 3D cameras

* Fix camera frames for real Orbbec Astra

* Fix Tf tree for Asus Xtion Pro

* Move pose of Asus Xtion Pro in Turtlebot stack

File: ca_description/urdf/sensors/lasers/astra.xacro (robot description, xacro)
@@ -3,12 +3,14 @@
 <xacro:include filename="$(find ca_description)/urdf/sensors/lasers/sim_3d_sensor.xacro"/>
 <!-- Orbbec Astra RGBD Camera -->
+<!-- https://github.com/orbbec/ros_astra_launch/blob/master/launch/includes/astra_frames.launch -->
 <xacro:property name="name" value="astra"/>
 <xacro:property name="parent" value="base_link"/>
-<xacro:property name="parent_link"    value="${parent}"/>
-<xacro:property name="link_name"      value="${name}_link"/>
-<xacro:property name="link_rgb"       value="${name}_rgb_frame"/>
-<xacro:property name="link_depth"     value="${name}_depth_frame"/>
-<xacro:property name="link_optical"   value="${name}_depth_optical_frame"/>
-<xacro:property name="optical_offset" value="0.01"/>
+<xacro:property name="parent_link"        value="${parent}"/>
+<xacro:property name="link_name"          value="${name}_link"/>
+<xacro:property name="link_rgb"           value="${name}_rgb_frame"/>
+<xacro:property name="link_rgb_optical"   value="${name}_rgb_optical_frame"/>
+<xacro:property name="link_depth"         value="${name}_depth_frame"/>
+<xacro:property name="link_depth_optical" value="${name}_depth_optical_frame"/>
+<xacro:property name="optical_rotation" value="${-pi/2} 0 ${-pi/2}"/>
 <joint name="${name}_joint" type="fixed">
   <origin xyz="${laser_origin}"/>
@@ -24,12 +26,18 @@
   </visual>
 </link>
-<joint name="${name}_optical_joint" type="fixed">
-  <origin xyz="0 ${optical_offset} 0" rpy="${-pi/2} 0 ${-pi/2}"/>
+<joint name="${name}_rgb_joint" type="fixed">
+  <origin xyz="0 -0.045 0"/>
   <parent link="${link_name}"/>
   <child link="${link_rgb}"/>
 </joint>
 <link name="${link_rgb}"/>
+<joint name="${name}_rgb_optical_joint" type="fixed">
+  <origin rpy="${optical_rotation}"/>
+  <parent link="${link_rgb}"/>
+  <child link="${link_rgb_optical}"/>
+</joint>
+<link name="${link_rgb_optical}"/>
 <joint name="${name}_depth_joint" type="fixed">
-  <origin rpy="${-pi/2} 0 ${-pi/2}"/>
+  <origin xyz="0 -0.02 0"/>
   <parent link="${link_name}"/>
   <child link="${link_depth}"/>
@@ -37,9 +45,9 @@
 <link name="${link_depth}"/>
   <joint name="${name}_depth_optical_joint" type="fixed">
-  <origin rpy="${-pi/2} 0 ${-pi/2}"/>
+  <origin rpy="${optical_rotation}"/>
   <parent link="${link_depth}"/>
-  <child link="${link_optical}"/>
+  <child link="${link_depth_optical}"/>
 </joint>
-<link name="${link_optical}"/>
+<link name="${link_depth_optical}"/>
 <xacro:sim_3d_sensor name="${name}" color="Gazebo/FlatBlack"/>
 </robot>

File: ca_description/urdf/sensors/lasers/xtion_pro.xacro (robot description, xacro)
@@ -9,29 +9,22 @@
 <xacro:property name="link_rgb"           value="${name}_rgb_frame"/>
 <xacro:property name="link_rgb_optical"   value="${name}_rgb_optical_frame"/>
+<xacro:property name="link_ir"            value="${name}_ir_frame"/>
+<xacro:property name="link_ir_optical"    value="${name}_ir_optical_frame"/>
 <xacro:property name="link_depth"         value="${name}_depth_frame"/>
 <xacro:property name="link_depth_optical" value="${name}_depth_optical_frame"/>
-<!-- Xacro properties -->
-<xacro:property name="xtion_pro_depth_rel_rgb_py" value="0.0270" />
-<xacro:property name="xtion_pro_cam_rel_rgb_py"   value="-0.0220" />
-<joint name="${name}_rgb_joint" type="fixed">
+<!-- This relates the IR sensor to the Xtion base link -->
+<!-- 4.8 cm because sensors are offset to right, from center -->
+<xacro:property name="ir_offset"        value="0.048"/>
+<!-- The measured distance from RGB lens back to IR lens, approx 2.5cm -->
+<xacro:property name="rgb_offset"       value="-0.025"/>
+<xacro:property name="optical_rotation" value="${-pi/2} 0 ${-pi/2}"/>
+<joint name="${name}_joint" type="fixed">
   <origin xyz="${laser_origin}"/>
-  <parent link="${parent}"/>
-  <child link="${link_rgb}" />
-</joint>
-<link name="${link_rgb}"/>
-<joint name="${name}_rgb_optical_joint" type="fixed">
-  <origin rpy="${-pi/2} 0 ${-pi/2}" />
-  <parent link="${link_rgb}" />
-  <child link="${link_rgb_optical}" />
-</joint>
-<link name="${link_rgb_optical}"/>
-<joint name="${name}_joint" type="fixed">
-  <origin xyz="0 ${xtion_pro_cam_rel_rgb_py} 0"/>
-  <parent link="${link_rgb}"/>
+  <parent link="${parent_link}"/>
   <child link="${link_name}"/>
 </joint>
 <link name="${link_name}">
   <visual>
-    <origin xyz="-0.015 0.0035 0.004"/>
+    <origin xyz="-0.015 0.0035 -0.01"/>
     <geometry>
       <mesh filename="package://ca_description/meshes/sensors/asus_xtion_pro_live.dae"/>
@@ -39,12 +32,28 @@
   </visual>
 </link>
+<!-- Xtion RGB sensor physical attachment -->
+<joint name="${name}_rgb_joint" type="fixed">
+  <origin xyz="0 ${rgb_offset} 0"/>
+  <parent link="${link_name}"/>
+  <child link="${link_rgb}" />
+</joint>
+<link name="${link_rgb}"/>
+<!-- Xtion RGB sensor frame -->
+<joint name="${name}_rgb_optical_joint" type="fixed">
+  <origin rpy="${optical_rotation}" />
+  <parent link="${link_rgb}" />
+  <child link="${link_rgb_optical}" />
+</joint>
+<link name="${link_rgb_optical}"/>
+<!-- Xtion IR sensor physical attachment -->
 <joint name="${name}_depth_joint" type="fixed">
-  <origin xyz="0 ${xtion_pro_depth_rel_rgb_py} 0"/>
+  <origin xyz="0 ${ir_offset} 0"/>
   <parent link="${link_rgb}" />
   <child link="${link_depth}"/>
 </joint>
 <link name="${link_depth}"/>
+<!-- Xtion IR sensor frame -->
 <joint name="${name}_depth_optical_joint" type="fixed">
-  <origin rpy="${-pi/2} 0 ${-pi/2}" />
+  <origin rpy="${optical_rotation}" />
   <parent link="${link_depth}" />
   <child link="${link_depth_optical}" />
